File: kicad/ATMega1608_Dev/ATMega1608_Dev.kicad_pcb (KiCad board)
At the start: 4 copper layers, 55.9 x 25.4 mm, 35 parts, among them J1 Alt Power, J101 GPIO2, J2 USB_B_Micro, J3 Comm, J4 GPIO1, J6 Power OUT, U1 TC1262-33, U2 FT232RQ, U3 ATMega1608_32

Commit message: Troubleshooting and diagnostic updates
Parts:
- C3, C4: footprint Capacitor_SMD:C_0805_2012Metric -> Capacitor_SMD:C_1206_3216Metric
- J2: footprint Connector_USB:USB_Micro-B_Amphenol_10103594-0001LF_Horizontal -> atmega1608_footprints:USB_Micro-B_Amphenol_10103594-0001LF_Horizontal
- moved C4 2.05 mm to (130.6, 60.7)
- moved C3 1.14 mm to (117.7, 59.7)
Routing:
- net Net-(J2-D+): track 14.6 -> 11.2 mm, vias 2 -> 0
- net Net-(U2-3V3Out): track 3.85 -> 5.83 mm
- net Net-(D2-A): track 45.3 -> 43.7 mm
- net /UPDI: track 35.2 -> 36.1 mm
- net Net-(J2-D-): track 12.0 -> 11.2 mm
- net Net-(U2-~{Reset}): track 4.03 -> 4.66 mm

Commit message: Move DIN R3 to top
Parts:
- R3: moved to F.Cu
Routing:
- net Net-(U2-TXD): track 2.68 -> 2.66 mm, vias 1 -> 0
- net /DIN: vias 1 -> 0
Changed lines of the file:
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@@
+    )
+  )
+  (footprint "Resistor_SMD:R_0805_2012Metric" (layer "F.Cu")
+    (at 126.746 69.596)
+    (descr "Resistor SMD 0805 (2012 Metric), square (rectangular) end terminal, IPC_7351 nominal, (Body size source: IPC-SM-782 page 72, https://www.pcb-3d.com/wordpress/wp-content/uploads/ipc-sm-782a_amendment_1_and_2.pdf), generated with kicad-footprint-generator")
+    (tags "resistor")
+    (property "Sheetfile" "ATMega1608_Dev.kicad_sch")
+    (property "Sheetname" "")
+    (property "ki_description" "Resistor")
+    (property "ki_keywords" "R res resistor")
+    (attr smd)
+    (fp_text reference "R3" (at -1.27 1.778) (layer "F.SilkS")
+        (effects (font (size 0.762 0.762) (thickness 0.127)))
+    )
+    (fp_text value "0Ω" (at 0 1.65) (layer "F.Fab")
+        (effects (font (size 0.762 0.762) (thickness 0.127)))
+    )
+    (fp_text user "${REFERENCE}" (at 0 0) (layer "F.Fab")
+        (effects (font (size 0.762 0.762) (thickness 0.127)))
+    )
+    (fp_line (start -0.227064 -0.735) (end 0.227064 -0.735)
+      (stroke (width 0.12) (type solid)) (layer "F.SilkS"))
+    (fp_line (start -0.227064 0.735) (end 0.227064 0.735)
+      (stroke (width 0.12) (type solid)) (layer "F.SilkS"))
+    (fp_line (start -1.68 -0.95) (end 1.68 -0.95)
+      (stroke (width 0.05) (type solid)) (layer "F.CrtYd"))
+    (fp_line (start -1.68 0.95) (end -1.68 -0.95)
+      (stroke (width 0.05) (type solid)) (layer "F.CrtYd"))
+    (fp_line (start 1.68 -0.95) (end 1.68 0.95)
+      (stroke (width 0.05) (type solid)) (layer "F.CrtYd"))
+    (fp_line (start 1.68 0.95) (end -1.68 0.95)
+      (stroke (width 0.05) (type solid)) (layer "F.CrtYd"))
+    (fp_line (start -1 -0.625) (end 1 -0.625)
+      (stroke (width 0.1) (type solid)) (layer "F.Fab"))
+    (fp_line (start -1 0.625) (end -1 -0.625)
+      (stroke (width 0.1) (type solid)) (layer "F.Fab"))
+    (fp_line (start 1 -0.625) (end 1 0.625)
+      (stroke (width 0.1) (type solid)) (layer "F.Fab"))
+    (fp_line (start 1 0.625) (end -1 0.625)
+      (stroke (width 0.1) (type solid)) (layer "F.Fab"))
+    (pad "1" smd roundrect (at -0.9125 0) (size 1.025 1.4) (layers "F.Cu" "F.Paste" "F.Mask") (roundrect_rratio 0.243902)
+      (net 42 "Net-(U2-TXD)") (pintype "passive"))
+    (pad "2" smd roundrect (at 0.9125 0) (size 1.025 1.4) (layers "F.Cu" "F.Paste" "F.Mask") (roundrect_rratio 0.243902)
+      (net 22 "/DIN") (pintype "passive"))
+    (model "${KICAD6_3DMODEL_DIR}/Resistor_SMD.3dshapes/R_0805_2012Metric.wrl"
+      (offset (xyz 0 0 0))
+      (scale (xyz 1 1 1))
+      (rotate (xyz 0 0 0))
     )
   )
@@
       (stroke (width 0.1) (type solid)) (fill solid) (layer "B.SilkS"))
   )
-  (footprint "Resistor_SMD:R_0805_2012Metric" (layer "B.Cu")
-    (at 126.746 69.596)
-    (descr "Resistor SMD 0805 (2012 Metric), square (rectangular) end terminal, IPC_7351 nominal, (Body size source: IPC-SM-782 page 72, https://www.pcb-3d.com/wordpress/wp-content/uploads/ipc-sm-782a_amendment_1_and_2.pdf), generated with kicad-footprint-generator")
-    (tags "resistor")
-    (property "Sheetfile" "ATMega1608_Dev.kicad_sch")
-    (property "Sheetname" "")
-    (property "ki_description" "Resistor")
-    (property "ki_keywords" "R res resistor")
-    (attr smd)
-    (fp_text reference "R3" (at 2.54 0) (layer "B.SilkS")
-        (effects (font (size 0.762 0.762) (thickness 0.127)) (justify mirror))
-    )
-    (fp_text value "0Ω" (at 0 -1.65) (layer "B.Fab")
-        (effects (font (size 0.762 0.762) (thickness 0.127)) (justify mirror))
-    )
-    (fp_text user "${REFERENCE}" (at 0 0) (layer "B.Fab")
-        (effects (font (size 0.762 0.762) (thickness 0.127)) (justify mirror))
-    )
-    (fp_line (start -0.227064 -0.735) (end 0.227064 -0.735)
-      (stroke (width 0.12) (type solid)) (layer "B.SilkS"))
-    (fp_line (start -0.227064 0.735) (end 0.227064 0.735)
-      (stroke (width 0.12) (type solid)) (layer "B.SilkS"))
-    (fp_line (start -1.68 -0.95) (end -1.68 0.95)
-      (stroke (width 0.05) (type solid)) (layer "B.CrtYd"))
-    (fp_line (start -1.68 0.95) (end 1.68 0.95)
-      (stroke (width 0.05) (type solid)) (layer "B.CrtYd"))
-    (fp_line (start 1.68 -0.95) (end -1.68 -0.95)
-      (stroke (width 0.05) (type solid)) (layer "B.CrtYd"))
-    (fp_line (start 1.68 0.95) (end 1.68 -0.95)
-      (stroke (width 0.05) (type solid)) (layer "B.CrtYd"))
-    (fp_line (start -1 -0.625) (end -1 0.625)
-      (stroke (width 0.1) (type solid)) (layer "B.Fab"))
-    (fp_line (start -1 0.625) (end 1 0.625)
-      (stroke (width 0.1) (type solid)) (layer "B.Fab"))
-    (fp_line (start 1 -0.625) (end -1 -0.625)
-      (stroke (width 0.1) (type solid)) (layer "B.Fab"))
-    (fp_line (start 1 0.625) (end 1 -0.625)
-      (stroke (width 0.1) (type solid)) (layer "B.Fab"))
-    (pad "1" smd roundrect (at -0.9125 0) (size 1.025 1.4) (layers "B.Cu" "B.Paste" "B.Mask") (roundrect_rratio 0.243902)
-      (net 42 "Net-(U2-TXD)") (pintype "passive"))
-    (pad "2" smd roundrect (at 0.9125 0) (size 1.025 1.4) (layers "B.Cu" "B.Paste" "B.Mask") (roundrect_rratio 0.243902)
-      (net 22 "/DIN") (pintype "passive"))
-    (model "${KICAD6_3DMODEL_DIR}/Resistor_SMD.3dshapes/R_0805_2012Metric.wrl"
-      (offset (xyz 0 0 0))
-      (scale (xyz 1 1 1))
-      (rotate (xyz 0 0 0))
-    )
-  )
   (footprint "Capacitor_SMD:C_1206_3216Metric" (layer "B.Cu")
     (at 117.729 59.69 180)
@@
   (segment (start 136.919422 70.5109) (end 137.070823 70.662301) (width 0.1524) (layer "F.Cu") (net 22))
   (segment (start 136.8825 70.473978) (end 136.919422 70.5109) (width 0.1524) (layer "F.Cu") (net 22))
+  (segment (start 127.6585 69.596) (end 128.6745 70.612) (width 0.1524) (layer "F.Cu") (net 22))
+  (segment (start 128.6745 70.612) (end 136.744478 70.612) (width 0.1524) (layer "F.Cu") (net 22))
   (segment (start 136.8825 69.215) (end 136.8825 70.473978) (width 0.1524) (layer "F.Cu") (net 22))
-  (via (at 136.919422 70.5109) (size 0.508) (drill 0.254) (layers "F.Cu" "B.Cu") (net 22))
-  (segment (start 136.818322 70.612) (end 136.919422 70.5109) (width 0.1524) (layer "B.Cu") (net 22))
-  (segment (start 127.6585 69.596) (end 128.6745 70.612) (width 0.1524) (layer "B.Cu") (net 22))
-  (segment (start 128.6745 70.612) (end 136.818322 70.612) (width 0.1524) (layer "B.Cu") (net 22))
+  (segment (start 136.744478 70.612) (end 136.8825 70.473978) (width 0.1524) (layer "F.Cu") (net 22))
   (segment (start 151.224897 67.977103) (end 150.241 68.961) (width 0.1524) (layer "F.Cu") (net 23))
   (segment (start 151.247695 67.977103) (end 151.224897 67.977103) (width 0.1524) (layer "F.Cu") (net 23))
@@
   (segment (start 124.0555 60.96) (end 123.003562 62.011938) (width 0.1524) (layer "B.Cu") (net 41))
   (segment (start 123.003562 62.011938) (end 123.003562 63.767351) (width 0.1524) (layer "B.Cu") (net 41))
-  (segment (start 127.496 68.124876) (end 127.496 67.7155) (width 0.1524) (layer "F.Cu") (net 42))
-  (segment (start 126.880795 68.740081) (end 127.496 68.124876) (width 0.1524) (layer "F.Cu") (net 42))
-  (via (at 126.880795 68.740081) (size 0.508) (drill 0.254) (layers "F.Cu" "B.Cu") (net 42))
-  (segment (start 125.8335 69.596) (end 125.984 69.596) (width 0.1524) (layer "B.Cu") (net 42))
-  (segment (start 126.024876 69.596) (end 126.880795 68.740081) (width 0.1524) (layer "B.Cu") (net 42))
-  (segment (start 125.984 69.596) (end 126.024876 69.596) (width 0.1524) (layer "B.Cu") (net 42))
+  (segment (start 125.984 69.596) (end 127.496 68.084) (width 0.1524) (layer "F.Cu") (net 42))
+  (segment (start 127.496 68.084) (end 127.496 67.7155) (width 0.1524) (layer "F.Cu") (net 42))
+  (segment (start 125.8335 69.596) (end 125.984 69.596) (width 0.1524) (layer "F.Cu") (net 42))
   (segment (start 131.4215 67.056) (end 130.8935 66.528) (width 0.1524) (layer "F.Cu") (net 43))
   (segment (start 130.8935 66.528) (end 129.1835 66.528) (width 0.1524) (layer "F.Cu") (net 43))
