File: kicad/ATMega1608_Dev/ATMega1608_Dev.kicad_sch (KiCad schematic)
At the start: 25 parts, among them J1 Alt Power, J2 USART-USB, J3 GPIO, J4 Power OUT, J5 GPIO2, U1 TC1262-33, U3 ATMega1608_32

Commit message: Adding a PCB release workflow
Parts:
- H1, H2, LG1, LG2, LG3: now left out of the parts list
